Commit message: slam

File: ros-pioneer3at/urdf/pioneer3at.xacro (robot description, xacro)
@@ -7,5 +7,5 @@
        name="pioneer3at">
 <!-- Chassis -->
-	<link name="Pioneer3AT/base_link">
+	<link name="base_link">
 		<visual>
 			<origin xyz="0 0 0.177" rpy="0 0 0"/>
@@ -32,5 +32,5 @@
 	<joint name="base_top_joint" type="fixed">
 		<origin xyz="0.003 0 0.274" rpy="0 0 0"/>
-		<parent link="Pioneer3AT/base_link"/>
+		<parent link="base_link"/>
 		<child link="top_plate"/>
 	</joint>
@@ -50,5 +50,5 @@
 	  <joint name="${prefix}_axle_joint" type="continuous">
 		  <origin xyz="${rx*0.135} ${ry*0.156} 0.111" rpy="0 0 0"/>
-		  <parent link="Pioneer3AT/base_link"/>
+		  <parent link="base_link"/>
 		  <child link="${prefix}_axle"/>
 		  <axis xyz="0 1 0" />
@@ -105,5 +105,5 @@
 	<joint name="front_sonar_joint" type="fixed">
 		<origin xyz="0.193 0 0.25" rpy="0 0 0"/>
-		<parent link="Pioneer3AT/base_link"/>
+		<parent link="base_link"/>
 		<child link="front_sonar"/>
 	</joint>
@@ -121,5 +121,5 @@
 	<joint name="rear_sonar_joint" type="fixed">
 		<origin xyz="-0.187 0 0.247" rpy="0 0 0"/>
-		<parent link="Pioneer3AT/base_link"/>
+		<parent link="base_link"/>
 		<child link="rear_sonar"/>
 	</joint>
@@ -138,5 +138,5 @@
 	  <joint name="Sonar_${id}_joint" type="fixed">
 		  <origin xyz="${px} ${py} 0.25" rpy="0 0 ${rz}"/>
-		  <parent link="Pioneer3AT/base_link"/>
+		  <parent link="base_link"/>
 		  <child link="Sonar_${id}"/>
 	  </joint>

Commit message: final

File: ros-pioneer3at/urdf/pioneer3at.xacro (robot description, xacro)
@@ -18,4 +18,14 @@
 		</visual>
 	</link>
+	<link name="OAK_D_link">
+		<visual>
+			<origin xyz="0.05 0.00 0.600" rpy="0 0 0"/>
+		</visual>
+	</link>
+	<joint name="OAK_camera_mount" type="fixed">
+		<origin xyz="0 0 0" rpy="0 0 0"/>
+		<parent link="base_link"/>
+		<child link="OAK_D_link"/>
+	</joint>
 <!-- Top -->
 	<link name="top_plate">
@@ -30,5 +40,5 @@
 			<origin xyz="0 0 0" rpy="0 0 0"/>
 			<geometry name="pioneer_geom">
-				<mesh filename="package://p3at_tutorial/meshes/top.dae"/>
+				<mesh filename="package://pioneer3at/meshes/top.dae"/>
 			</geometry>
 			<material name="TopBlack">
